Commit message: chore: add dummy for simulate base_link inertia and new rviz configurations

File: robots_description/differential/urdf/diff.description.urdf.xacro (robot description, xacro)
@@ -1,25 +1,23 @@
 <?xml version="1.0"?>
-<!--
-Copied from ROS2 control demos:
-https://github.com/ros-controls/ros2_control_demos/blob/humble/ros2_control_demo_description/diffbot/urdf/diffbot_description.urdf.xacro
--->
 <robot xmlns:xacro="http://www.ros.org/wiki/xacro">
     <xacro:macro name="diffbot" params="prefix">
         <!-- Constants for robot dimensions -->
         <xacro:property name="PI" value="3.1415926535897931" />
-        <xacro:property name="base_mass" value="0.3" /> <!-- arbitrary value for base mass -->
+        <xacro:property name="base_mass" value="0.3" />
         <xacro:property name="base_width" value="0.1" />
         <xacro:property name="base_length" value="0.1" />
         <xacro:property name="base_height" value="0.05" />
-        <xacro:property name="wheel_mass" value="0.3" /> <!-- arbitrary value for wheel mass -->
+        <xacro:property name="wheel_mass" value="0.3" />
         <xacro:property name="wheel_len" value="0.020" />
         <xacro:property name="wheel_radius" value="0.015" />
-        <xacro:property name="caster_wheel_mass" value="0.1" /> <!-- arbitrary value for caster wheel
-        mass -->
+        <xacro:property name="caster_wheel_mass" value="0.1" />
         <xacro:property name="caster_wheel_radius" value="0.015" />
-        <xacro:property name="z_offset" value="-${base_height/2}" /> <!-- Space btw top of beam and
-        the each joint -->
-        <!-- Base Link -->
+        <xacro:property name="z_offset" value="-${base_height/2}" />
+        <!-- Modified Base Link -->
         <link name="${prefix}base_link">
+            <!-- No visual, collision, or inertial components needed -->
+        </link>
+        <!-- Dummy Link -->
+        <link name="${prefix}base_dummy_link">
             <collision>
                 <origin xyz="0 0 0" rpy="0 0 0" />
@@ -46,4 +44,11 @@
             </inertial>
         </link>
+        <!-- Joint Connecting Dummy Link to Base Link -->
+        <joint name="${prefix}base_dummy_joint" type="fixed">
+            <parent link="${prefix}base_link" />
+            <child link="${prefix}base_dummy_link" />
+            <origin xyz="0 0 0" rpy="0 0 0" />
+        </joint>
+        <!-- Rest of your robot definition -->
         <joint name="${prefix}left_wheel_joint" type="continuous">
             <parent link="${prefix}base_link" />
